File: Board Layout/Coffee.sch (KiCad schematic (older format))
At the start: 15 parts, among them CON1 AVR-JTAG-10, U1 ISO7341FC, U1 STM32F407VGTx, U2 ISO7341FC

Commit message: Replace Coffee.sch
Parts:
- removed C?: 0.1µ, symbol C_Small
- removed CON1: AVR-JTAG-10, AVR-JTAG-10, symbol AVR-JTAG-10
- added C3: 0.1µ, Capacitors_SMD:C_1206_HandSoldering, symbol C_Small
- added JTAG: JTAG-20, symbol JTAG-20
- added R10, R5, R6, R7, R8, R9: 470, symbol R
- C1, C2: footprint (none) -> Capacitors_SMD:C_1206_HandSoldering
- C4: renamed from C?; footprint (none) -> Capacitors_SMD:C_1206_HandSoldering
- J1: renamed from J?; value Conn_02x04_Odd_Even -> Conn_PB; footprint (none) -> Pin_Headers:Pin_Header_Straight_2x04_Pitch1.27mm
- J2: renamed from J?; value Conn_02x04_Odd_Even -> Conn_LCD; footprint (none) -> Pin_Headers:Pin_Header_Straight_2x04_Pitch1.27mm
- J3: renamed from J?; value Conn_01x04 -> USART; footprint (none) -> Pin_Headers:Pin_Header_Straight_1x04_Pitch1.27mm
- R1, R2, R3, R4: footprint (none) -> Resistors_SMD:R_0805_HandSoldering
- U1: footprint LQFP100 -> Housings_QFP:LQFP-100_14x14mm_Pitch0.5mm
- renumbered U1 to U3
Connections:
- net labels added: 2, 3, 4
- net labels removed: 3.3v, SPI3_MISO, SPI3_MOSI, SPI3_SCK
- wire segments 130 -> 142
Other:
- moved on the sheet: C1, C2, C4, J1, J2
